Commit message: camera try #1

File: src/robot_sim/model_description/models/Qbert/qbert.urdf (robot description, URDF)
Before this commit: robot Qbert, 4 links, 3 joints
Links:
- removed link camera
- added link camera_link, mass 1e-9
- added link camera_link_optical
- link base: geometry collision mesh filename=package://model_description/models/Qbert/assets/merged/base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; visual mesh filename=package://model_description/models/Qbert/assets/merged/base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
- link drum_assembly: geometry collision mesh filename=package://model_description/models/Qbert/assets/merged/drum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; visual mesh filename=package://model_description/models/Qbert/assets/merged/drum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
- link part_1: geometry collision mesh filename=package://model_description/models/Qbert/assets/merged/part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; visual mesh filename=package://model_description/models/Qbert/assets/merged/part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
Joints:
- removed joint camera_frame
- added joint camera_joint: type fixed, parent drum_assembly, child camera_link, origin xyz=-0.127664 0.127727 0.345195 rpy=1.46442 2.59821e-16 0.785398, axis 0 0 0
- added joint camera_optical_joint: type fixed, parent camera_link, child camera_link_optical, origin xyz=0 0 0 rpy=${-pi/2} 0 ${-pi/2}

Commit message: working cam

File: src/robot_sim/model_description/models/Qbert/qbert.urdf (robot description, URDF)
Before this commit: robot Qbert, 5 links, 4 joints
Links:
- removed link camera_link_optical
- added link camera_optical_link
Joints:
- joint camera_optical_joint: child camera_link_optical -> camera_optical_link
